Commit message: update

File: models/franka_panda/panda_with_stick.urdf (robot description, URDF)
Before this commit: robot panda, 14 links, 13 joints
Links:
- added link sticktarget, mass 0.0
- link stick: geometry collision box size=0.075 0.003 0.003; visual box size=0.075 0.003 0.003
Joints:
- added joint sticktarget_hand: type fixed, parent stick, child sticktarget, origin xyz=-0.075 0 0 rpy=0 0 0
- joint stick_finger_joint: origin xyz=0.0375 -0.015 0.05 rpy=0 0 0 -> xyz=0 0 0.05 rpy=0 0 0
