Commit message: update move fcts and add robot urdfs

File: models/franka_panda/panda_stick_right_back.urdf (robot description, URDF)
Before this commit: robot panda, 15 links, 14 joints
Links:
- link stick: geometry collision box size=-0.075 0.003 0.003; visual box size=-0.075 0.003 0.003
Joints:
- joint stick_finger_joint: origin xyz=0 0 0.05 rpy=0 0 0 -> xyz=0 -0.005 0.05 rpy=0 0 0
- joint sticktarget_hand: origin xyz=-0.075 0 0 rpy=0 0 0 -> xyz=0.075 0 0 rpy=0 0 0
