Commit message: extend sticks from 7.5 to 10cm

File: models/franka_panda/panda_stick_left_back.urdf (robot description, URDF)
Before this commit: robot panda, 15 links, 14 joints
Links:
- link stick: geometry collision box size=-0.10 0.003 0.003; visual box size=-0.10 0.003 0.003
Joints:
- joint sticktarget_hand: origin xyz=0.075 0 0 rpy=0 0 0 -> xyz=0.10 0 0 rpy=0 0 0

File: models/franka_panda/panda_stick_left_front.urdf (robot description, URDF)
Before this commit: robot panda, 15 links, 14 joints
Links:
- link stick: geometry collision box size=0.10 0.003 0.003; visual box size=0.10 0.003 0.003
Joints:
- joint sticktarget_hand: origin xyz=-0.075 0 0 rpy=0 0 0 -> xyz=-0.10 0 0 rpy=0 0 0

File: models/franka_panda/panda_stick_left_top.urdf (robot description, URDF)
Before this commit: robot panda, 15 links, 14 joints
Links:
- link stick: geometry collision box size=0.003 0.003 0.10; visual box size=0.003 0.003 0.10
Joints:
- joint sticktarget_hand: origin xyz=0 0 0.075 rpy=0 0 0 -> xyz=0 0 0.10 rpy=0 0 0

File: models/franka_panda/panda_stick_right_back.urdf (robot description, URDF)
Before this commit: robot panda, 15 links, 14 joints
Links:
- link stick: geometry collision box size=-0.10 0.003 0.003; visual box size=-0.10 0.003 0.003
Joints:
- joint sticktarget_hand: origin xyz=0.075 0 0 rpy=0 0 0 -> xyz=0.10 0 0 rpy=0 0 0

File: models/franka_panda/panda_stick_right_front.urdf (robot description, URDF)
Before this commit: robot panda, 15 links, 14 joints
Links:
- link stick: geometry collision box size=0.10 0.003 0.003; visual box size=0.10 0.003 0.003
Joints:
- joint sticktarget_hand: origin xyz=-0.075 0 0 rpy=0 0 0 -> xyz=-0.10 0 0 rpy=0 0 0

File: models/franka_panda/panda_stick_right_top.urdf (robot description, URDF)
Before this commit: robot panda, 15 links, 14 joints
Links:
- link stick: geometry collision box size=0.003 0.003 0.10; visual box size=0.003 0.003 0.10
Joints:
- joint sticktarget_hand: origin xyz=0 0 0.075 rpy=0 0 0 -> xyz=0 0 0.10 rpy=0 0 0

Commit message: resize stick length, add orientation to tower

File: models/franka_panda/panda_stick_left_back.urdf (robot description, URDF)
Before this commit: robot panda, 15 links, 14 joints
Links:
- added link cam, mass 0.1; collision box size=0.03 0.1 0.03; visual box size=0.03 0.1 0.03
- link stick: geometry collision box size=-0.15 0.003 0.003; visual box size=-0.15 0.003 0.003
Joints:
- added joint cam_joint: type fixed, parent panda_hand, child cam, origin xyz=0 -0.005 0.05 rpy=0 0 0
- joint sticktarget_hand: origin xyz=0.10 0 0 rpy=0 0 0 -> xyz=0.15 0 0 rpy=0 0 0

File: models/franka_panda/panda_stick_left_front.urdf (robot description, URDF)
Before this commit: robot panda, 15 links, 14 joints
Links:
- added link cam, mass 0.1; collision box size=0.03 0.1 0.03; visual box size=0.03 0.1 0.03
- link stick: geometry collision box size=0.15 0.003 0.003; visual box size=0.15 0.003 0.003
Joints:
- added joint cam_joint: type fixed, parent panda_hand, child cam, origin xyz=0 -0.005 0.05 rpy=0 0 0
- joint sticktarget_hand: origin xyz=-0.10 0 0 rpy=0 0 0 -> xyz=-0.15 0 0 rpy=0 0 0

File: models/franka_panda/panda_stick_left_top.urdf (robot description, URDF)
Before this commit: robot panda, 15 links, 14 joints
Links:
- added link cam, mass 0.1; collision box size=0.03 0.1 0.03; visual box size=0.03 0.1 0.03
Joints:
- added joint cam_joint: type fixed, parent panda_hand, child cam, origin xyz=0 -0.005 0.05 rpy=0 0 0

File: models/franka_panda/panda_stick_right_back.urdf (robot description, URDF)
Before this commit: robot panda, 15 links, 14 joints
Links:
- added link cam, mass 0.1; collision box size=0.03 0.1 0.03; visual box size=0.03 0.1 0.03
- link stick: geometry collision box size=-0.15 0.003 0.003; visual box size=-0.15 0.003 0.003
Joints:
- added joint cam_joint: type fixed, parent panda_hand, child cam, origin xyz=0 -0.005 0.05 rpy=0 0 0
- joint sticktarget_hand: origin xyz=0.10 0 0 rpy=0 0 0 -> xyz=0.15 0 0 rpy=0 0 0

File: models/franka_panda/panda_stick_right_front.urdf (robot description, URDF)
Before this commit: robot panda, 15 links, 14 joints
Links:
- added link cam, mass 0.1; collision box size=0.03 0.1 0.03; visual box size=0.03 0.1 0.03
- link stick: geometry collision box size=0.15 0.003 0.003; visual box size=0.15 0.003 0.003
Joints:
- added joint cam_joint: type fixed, parent panda_hand, child cam, origin xyz=0 -0.005 0.05 rpy=0 0 0
- joint sticktarget_hand: origin xyz=-0.10 0 0 rpy=0 0 0 -> xyz=-0.15 0 0 rpy=0 0 0

File: models/franka_panda/panda_stick_right_top.urdf (robot description, URDF)
Before this commit: robot panda, 15 links, 14 joints
Links:
- added link cam, mass 0.1; collision box size=0.03 0.1 0.03; visual box size=0.03 0.1 0.03
Joints:
- added joint cam_joint: type fixed, parent panda_hand, child cam, origin xyz=0 -0.005 0.05 rpy=0 0 0
